File: Hardware/SparkFun_MicroMod_DA16200_Function.brd (EAGLE design)
At the start: 65 x 38 mm, 57 parts, among them J1 MICROMOD_STANDARD, J2 CORTEX_JTAG_DEBUG, U1 DA16200MOD, U2 CH340E_MSOP10, U3 3.3V, U4 EEPROM

Commit message: Updates the design to use the Micromod-function device in the official SFE Eagle Libs
Parts:
- J1: value MICROMOD_STANDARD -> MICROMOD_FUNCTION_STANDARD; device SparkFun-MicroMod-Function:M.2-CARD-E-22_FUNCTION_STANDARD -> SparkFun-MicroMod:M.2-CARD-E-22_FUNCTION_STANDARD
Changed lines of the file:
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@@
 <?xml version="1.0" encoding="utf-8"?>
 <!DOCTYPE eagle SYSTEM "eagle.dtd">
-<eagle version="9.6.2">
+<eagle version="9.5.1">
 <drawing>
 <settings>
@@
 </autorouter>
 <elements>
-<element name="J1" library="SparkFun-MicroMod-Function" package="M.2-CARD-E-22_FUNCTION_STANDARD" value="MICROMOD_STANDARD" x="0" y="19" smashed="yes" rot="R270"/>
+<element name="J1" library="SparkFun-MicroMod" package="M.2-CARD-E-22_FUNCTION_STANDARD" value="MICROMOD_FUNCTION_STANDARD" x="0" y="19" smashed="yes" rot="R270"/>
 <element name="U3" library="SparkFun-IC-Power" package="SOT23-5" value="3.3V" x="15.748" y="27.559" smashed="yes" rot="R270">
 <attribute name="NAME" x="17.907" y="29.337" size="0.6096" layer="25" ratio="20" rot="R270"/>
